Commit message: feat(arm-cell): publish v0.2.0 public package

File: infra/isaac_sim/assets/third_party/robotiq_description/urdf/robotiq_2f_85_macro.urdf.xacro (robot description, xacro)
@@ -1,275 +1 @@
-<?xml version="1.0"?>
-<robot xmlns:xacro="http://wiki.ros.org/xacro" name="robotiq_gripper">
-    <xacro:macro name="robotiq_gripper" params="
-        name
-        prefix
-        parent
-        mesh_dir
-        *origin
-        sim_gazebo:=false
-        sim_isaac:=false
-        isaac_joint_commands:=/isaac_joint_commands
-        isaac_joint_states:=/isaac_joint_states
-        use_fake_hardware:=false
-        mock_sensor_commands:=false
-        com_port:=/dev/ttyUSB0
-        baudrate:=115200
-        gripper_speed_multiplier:=1.0
-        gripper_force_multiplier:=0.5
-        gripper_max_speed:=0.150
-        gripper_max_force:=235.0
-        gripper_closed_position:=0.7929">
-        <link name="${prefix}robotiq_85_base_link">
-            <visual>
-                <geometry>
-                    <mesh filename="${mesh_dir}/visual/2f_85/robotiq_base.dae"/>
-                </geometry>
-            </visual>
-            <collision>
-                <geometry>
-                    <mesh filename="${mesh_dir}/collision/2f_85/robotiq_base.stl" />
-                </geometry>
-            </collision>
-            <inertial>
-                <origin xyz="0.0 2.274e-05 0.03232288" rpy="0 0 0" />
-                <mass value="6.6320197e-01" />
-                <inertia ixx="5.1617816e-04" iyy="5.8802208e-04" izz="3.9462776e-04" ixy="2.936e-8" ixz="0.0" iyz="-3.2296e-7" />
-            </inertial>
-        </link>
-        <link name="${prefix}robotiq_85_left_knuckle_link">
-            <visual>
-                <geometry>
-                    <mesh filename="${mesh_dir}/visual/2f_85/left_knuckle.dae" />
-                </geometry>
-            </visual>
-            <collision>
-                <geometry>
-                    <mesh filename="${mesh_dir}/collision/2f_85/left_knuckle.stl" />
-                </geometry>
-            </collision>
-            <inertial>
-                <origin xyz="0.01213197 0.0002 -0.00058647" rpy="0 0 0" />
-                <mass value="1.384773208e-02" />
-                <inertia ixx="3.5232e-7" iyy="2.31944e-6" izz="2.23136e-6" ixy="0.0" ixz="1.1744e-7" iyz="0" />
-            </inertial>
-        </link>
-        <link name="${prefix}robotiq_85_right_knuckle_link">
-            <visual>
-                <geometry>
-                    <mesh filename="${mesh_dir}/visual/2f_85/right_knuckle.dae" />
-                </geometry>
-            </visual>
-            <collision>
-                <geometry>
-                    <mesh filename="${mesh_dir}/collision/2f_85/right_knuckle.stl" />
-                </geometry>
-            </collision>
-            <inertial>
-                <origin xyz="-0.01213197 0.0002 -0.00058647" rpy="0 0 0" />
-                <mass value="1.384773208e-02" />
-                <inertia ixx="3.5232e-7" iyy="2.31944e-6" izz="2.23136e-6" ixy="0.0" ixz="-1.1744e-7" iyz="0.0" />
-            </inertial>
-        </link>
-        <link name="${prefix}robotiq_85_left_finger_link">
-            <visual>
-                <geometry>
-                    <mesh filename="${mesh_dir}/visual/2f_85/left_finger.dae" />
-                </geometry>
-            </visual>
-            <collision>
-                <geometry>
-                    <mesh filename="${mesh_dir}/collision/2f_85/left_finger.stl" />
-                </geometry>
-            </collision>
-            <inertial>
-                <origin xyz="0.00346899 -0.00079447 0.01867121" rpy="0 0 0" />
-                <mass value="4.260376752e-02" />
-                <inertia ixx="1.385792000000000e-05" iyy="1.183208e-05" izz="5.19672e-06" ixy="0.0" ixz="-2.17264e-06" iyz="0.0" />
-            </inertial>
-        </link>
-        <link name="${prefix}robotiq_85_right_finger_link">
-            <visual>
-                <geometry>
-                    <mesh filename="${mesh_dir}/visual/2f_85/right_finger.dae" />
-                </geometry>
-            </visual>
-            <collision>
-                <geometry>
-                    <mesh filename="${mesh_dir}/collision/2f_85/right_finger.stl" />
-                </geometry>
-            </collision>
-            <inertial>
-                <origin xyz="-0.00346899 -5.53e-06 0.01867121" rpy="0 0 0" />
-                <mass value="4.260376752000000e-02" />
-                <inertia ixx="1.385792e-05" iyy="1.183208e-05" izz="5.19672e-06" ixy="0.0" ixz="2.17264e-06" iyz="0.0" />
-            </inertial>
-        </link>
-        <link name="${prefix}robotiq_85_left_inner_knuckle_link">
-            <visual>
-                <geometry>
-                    <mesh filename="${mesh_dir}/visual/2f_85/left_inner_knuckle.dae" />
-                </geometry>
-            </visual>
-            <collision>
-                <geometry>
-                    <mesh filename="${mesh_dir}/collision/2f_85/left_inner_knuckle.stl" />
-                </geometry>
-            </collision>
-            <inertial>
-                <origin xyz="0.01897699 0.00015001 0.02247101" rpy="0 0 0" />
-                <mass value="2.969376448e-02" />
-                <inertia ixx="9.57136e-06" iyy="8.69056e-06" izz="8.19144e-06" ixy="0.0" ixz="-3.93424e-06" iyz="0.0" />
-            </inertial>
-        </link>
-        <link name="${prefix}robotiq_85_right_inner_knuckle_link">
-            <visual>
-                <geometry>
-                    <mesh filename="${mesh_dir}/visual/2f_85/right_inner_knuckle.dae" />
-                </geometry>
-            </visual>
-            <collision>
-                <geometry>
-                    <mesh filename="${mesh_dir}/collision/2f_85/right_inner_knuckle.stl" />
-                </geometry>
-            </collision>
-            <inertial>
-                <origin xyz="-0.01926824 5.001e-05 0.02222178" rpy="0 0 0" />
-                <mass value="2.969376448e-02" />
-                <inertia ixx="9.42456e-06" iyy="8.69056e-06" izz="8.33824e-06" ixy="0.0" ixz="3.9636e-06" iyz="0.0" />
-            </inertial>
-        </link>
-        <link name="${prefix}robotiq_85_left_finger_tip_link">
-            <visual>
-                <geometry>
-                    <mesh filename="${mesh_dir}/visual/2f_85/left_finger_tip.dae" />
-                </geometry>
-            </visual>
-            <collision>
-                <geometry>
-                    <mesh filename="${mesh_dir}/collision/2f_85/left_finger_tip.stl" />
-                </geometry>
-                <surface>
-                    <friction>
-                    <ode>
-                        <mu1>100000.0</mu1>
-                        <mu2>100000.0</mu2>
-                    </ode>
-                    </friction>
-                    <contact>
-                    <ode>
-                        <kp>1e+5</kp>
-                        <kd>1</kd>
-                        <soft_cfm>0</soft_cfm>
-                        <soft_erp>0.2</soft_erp>
-                        <minDepth>0.002</minDepth>
-                        <maxVel>0</maxVel>
-                    </ode>
-                    </contact>
-                </surface>
-            </collision>
-            <inertial>
-                <origin xyz="-0.01456706 -0.0008 0.01649701" rpy="0 0 0" />
-                <mass value="4.268588744e-02" />
-                <inertia ixx="1.048152e-05" iyy="1.197888e-05" izz="4.22784e-06" ixy="0.0" ixz="3.5232e-6" iyz="0.0" />
-            </inertial>
-        </link>
-        <link name="${prefix}robotiq_85_right_finger_tip_link">
-            <visual>
-                <geometry>
-                    <mesh filename="${mesh_dir}/visual/2f_85/right_finger_tip.dae" />
-                </geometry>
-            </visual>
-            <collision>
-                <geometry>
-                    <mesh filename="${mesh_dir}/collision/2f_85/right_finger_tip.stl" />
-                </geometry>
-                <surface>
-                    <friction>
-                    <ode>
-                        <mu1>100000.0</mu1>
-                        <mu2>100000.0</mu2>
-                    </ode>
-                    </friction>
-                    <contact>
-                    <ode>
-                        <kp>1e+5</kp>
-                        <kd>1</kd>
-                        <soft_cfm>0</soft_cfm>
-                        <soft_erp>0.2</soft_erp>
-                        <minDepth>0.002</minDepth>
-                        <maxVel>0</maxVel>
-                    </ode>
-                    </contact>
-                </surface>
-            </collision>
-            <inertial>
-                <origin xyz="0.01456706 5e-05 0.01649701" rpy="0 0 0" />
-                <mass value="4.268588744e-02" />
-                <inertia ixx="1.048152e-05" iyy="1.197888e-05" izz="4.22784e-06" ixy="0.0" ixz="-3.5232e-06" iyz="0.0" />
-            </inertial>
-        </link>
-        <joint name="${prefix}robotiq_85_base_joint" type="fixed">
-            <parent link="${parent}" />
-            <child link="${prefix}robotiq_85_base_link" />
-            <xacro:insert_block name="origin" />
-        </joint>
-        <joint name="${prefix}robotiq_85_left_knuckle_joint" type="revolute">
-            <parent link="${prefix}robotiq_85_base_link" />
-            <child link="${prefix}robotiq_85_left_knuckle_link" />
-            <axis xyz="0 -1 0" />
-            <origin xyz="0.03060114 0.0 0.05490452" rpy="0 0 0" />
-            <limit lower="0.0" upper="0.8" velocity="0.5" effort="50" />
-        </joint>
-        <joint name="${prefix}robotiq_85_right_knuckle_joint" type="revolute">
-            <parent link="${prefix}robotiq_85_base_link" />
-            <child link="${prefix}robotiq_85_right_knuckle_link" />
-            <axis xyz="0 -1 0" />
-            <origin xyz="-0.03060114 0.0 0.05490452" rpy="0 0 0" />
-            <limit lower="-0.8" upper="0.0" velocity="0.5" effort="50" />
-            <mimic joint="${prefix}robotiq_85_left_knuckle_joint" multiplier="-1" />
-        </joint>
-        <joint name="${prefix}robotiq_85_left_finger_joint" type="fixed">
-            <parent link="${prefix}robotiq_85_left_knuckle_link" />
-            <child link="${prefix}robotiq_85_left_finger_link" />
-            <origin xyz="0.03152616 0.0 -0.00376347" rpy="0 0 0" />
-        </joint>
-        <joint name="${prefix}robotiq_85_right_finger_joint" type="fixed">
-            <parent link="${prefix}robotiq_85_right_knuckle_link" />
-            <child link="${prefix}robotiq_85_right_finger_link" />
-            <origin xyz="-0.03152616 0.0 -0.00376347" rpy="0 0 0" />
-        </joint>
-        <joint name="${prefix}robotiq_85_left_inner_knuckle_joint" type="revolute">
-            <parent link="${prefix}robotiq_85_base_link" />
-            <child link="${prefix}robotiq_85_left_inner_knuckle_link" />
-            <axis xyz="0 -1 0" />
-            <origin xyz="0.0127 0.0 0.06142" rpy="0 0 0" />
-            <mimic joint="${prefix}robotiq_85_left_knuckle_joint"
-            multiplier="1" />
-            <limit lower="0.0" upper="0.8" velocity="0.5" effort="50" />
-        </joint>
-        <joint name="${prefix}robotiq_85_right_inner_knuckle_joint" type="revolute">
-            <parent link="${prefix}robotiq_85_base_link" />
-            <child link="${prefix}robotiq_85_right_inner_knuckle_link" />
-            <axis xyz="0 -1 0" />
-            <origin xyz="-0.0127 0.0 0.06142" rpy="0 0 0" />
-            <mimic joint="${prefix}robotiq_85_left_knuckle_joint" multiplier="-1" />
-            <limit lower="-0.8" upper="0.0" velocity="0.5" effort="50" />
-        </joint>
-        <joint name="${prefix}robotiq_85_left_finger_tip_joint" type="revolute">
-            <parent link="${prefix}robotiq_85_left_finger_link" />
-            <child link="${prefix}robotiq_85_left_finger_tip_link" />
-            <axis xyz="0 -1 0" />
-            <origin xyz="0.00563134 0.0 0.04718515" rpy="0 0 0" />
-            <mimic joint="${prefix}robotiq_85_left_knuckle_joint" multiplier="-1" />
-            <limit lower="-0.8" upper="0.0" velocity="0.5" effort="50" />
-        </joint>
-        <joint name="${prefix}robotiq_85_right_finger_tip_joint" type="revolute">
-            <parent link="${prefix}robotiq_85_right_finger_link" />
-            <child link="${prefix}robotiq_85_right_finger_tip_link" />
-            <axis xyz="0 -1 0" />
-            <origin xyz="-0.00563134 0.0 0.04718515" rpy="0 0 0" />
-            <mimic joint="${prefix}robotiq_85_left_knuckle_joint" />
-            <limit lower="0.0" upper="0.8" velocity="0.5" effort="50" />
-        </joint>
-    </xacro:macro>
-</robot>
+../../../../../../ros2_ws/src/arm_cell/arm_cell_description/urdf/robotiq_2f_85_macro.urdf.xacro

File: infra/isaac_sim/assets/urdf/adapters/m0609_tool_adapter.xacro (robot description, xacro)
@@ -1,32 +1 @@
-<?xml version="1.0"?>
-<robot xmlns:xacro="http://www.ros.org/wiki/xacro">
-    <!--
-      SF-Twin standard tool adapter
-      Robot side:
-          M0609 tool0
-      Tool side:
-          tool_mount
-      Vendor-specific grippers must attach to tool_mount,
-      not directly to tool0.
-    -->
-    <xacro:macro name="m0609_tool_adapter" params="
-        parent
-        adapter_link:=sf_tool_adapter
-        mount_link:=tool_mount
-        xyz:='0 0 0'
-        rpy:='0 0 0'
-    ">
-        <link name="${adapter_link}"/>
-        <joint name="${parent}_to_${adapter_link}" type="fixed">
-            <parent link="${parent}"/>
-            <child link="${adapter_link}"/>
-            <origin xyz="${xyz}" rpy="${rpy}"/>
-        </joint>
-        <link name="${mount_link}"/>
-        <joint name="${adapter_link}_to_${mount_link}" type="fixed">
-            <parent link="${adapter_link}"/>
-            <child link="${mount_link}"/>
-            <origin xyz="0 0 0" rpy="0 0 0"/>
-        </joint>
-    </xacro:macro>
-</robot>
+../../../../../ros2_ws/src/arm_cell/arm_cell_description/urdf/m0609_tool_adapter.xacro

File: infra/isaac_sim/assets/urdf/robots/m0609_macro.xacro (robot description, xacro)
@@ -1,248 +1 @@
-<?xml version="1.0"?>
-<robot xmlns:xacro="http://www.ros.org/wiki/xacro">
-    <xacro:macro name="m0609_robot" params="mesh_dir">
-	    <!-- Base Link -->
-	    <link name="base_link">
-		<inertial>
-		    <mass value="3.18"/>
-		    <origin xyz="-2.8e-05 -0.006045 0.038403"/>
-		    <inertia ixx="0.017789" ixy="-7.4356e-06" ixz="3.0378e-06" iyy="0.011135" iyz="-0.00029038" izz="0.020054"/>
-		</inertial>
-		<collision>
-		    <origin rpy="0 0 0" xyz="0 0 0" />
-		    <geometry>
-		        <mesh filename="${mesh_dir}/m0609_collision/MF0609_0_0.dae" scale="0.001 0.001 0.001" />
-		    </geometry>
-		</collision>
-		<visual>
-		    <origin rpy="0 0 0" xyz="0 0 0" />
-		    <geometry>
-		        <mesh filename="${mesh_dir}/m0609_white/MF0609_0_0.dae" scale="0.001 0.001 0.001" />
-		    </geometry>
-		</visual>
-	    </link>
-	    <link name="base"/>
-	    <joint name="base_link-base" type="fixed">
-		<origin rpy="0 0 0" xyz="0 0 0.450"/>
-		<parent link="base_link"/>
-		<child link="base"/>
-	    </joint>
-	    <!-- Joint 1 -->
-	    <joint name="joint_1" type="revolute">
-		<parent link="base_link" />
-		<child link="link_1" />
-		<origin rpy="0 0 0" xyz="0 0 0.1345" />
-		<axis xyz="0 0 1" />
-		<limit effort="9600" lower="-6.2832" upper="6.2832" velocity="2.618"/>
-		<dynamics friction="0.5" damping="500.0" stiffness="10000.0"/>
-	    </joint>
-	    <!-- Link 1 -->
-	    <link name="link_1">
-		<inertial>
-		    <mass value="5.02"/>
-		    <origin xyz="7.2e-05 0.036227 -0.003417"/>
-		    <inertia ixx="0.026195" ixy="2.3904e-05" ixz="-1.3319e-05" iyy="0.016899" iyz="-0.00071987" izz="0.022944"/>
-		</inertial>
-		<collision>
-		    <origin rpy="0 0 0" xyz="0 0 0" />
-		    <geometry>
-		        <mesh filename="${mesh_dir}/m0609_collision/MF0609_1_0.dae" scale="0.001 0.001 0.001" />
-		    </geometry>
-		</collision>
-		<visual>
-		    <origin rpy="0 0 0" xyz="0 0 0" />
-		    <geometry>
-		        <mesh filename="${mesh_dir}/m0609_white/MF0609_1_0.dae" scale="0.001 0.001 0.001" />
-		    </geometry>
-		</visual>
-	    </link>
-	    <!-- Joint 2 -->
-	    <joint name="joint_2" type="revolute">
-		<parent link="link_1" />
-		<child link="link_2" />
-		<origin rpy="0 -1.571 -1.571" xyz="0 0.0062 0" />
-		<axis xyz="0 0 1" />
-		<limit effort="9600" lower="-6.2832" upper="6.2832" velocity="2.618"/>
-		<dynamics friction="0.5" damping="500.0" stiffness="10000.0"/>
-	    </joint>
-	    <!-- Link 2 -->
-	    <link name="link_2">
-		<inertial>
-		    <mass value="8.04"/>
-		    <origin xyz="0.20447 2.6e-05 0.16005"/>
-		    <inertia ixx="0.026743" ixy="-0.00019461" ixz="-0.00058734" iyy="0.30084" iyz="-6.7892e-06" izz="0.29898"/>
-		</inertial>
-		<collision>
-		    <origin rpy="0 0 0" xyz="0 0 0" />
-		    <geometry>
-		        <mesh filename="${mesh_dir}/m0609_collision/MF0609_2_0.dae" scale="0.001 0.001 0.001" />
-		    </geometry>
-		</collision>
-		<visual>
-		    <origin rpy="0 0 0" xyz="0 0 0" />
-		    <geometry>
-		        <mesh filename="${mesh_dir}/m0609_white/MF0609_2_0.dae" scale="0.001 0.001 0.001" />
-		    </geometry>
-		</visual>
-		<collision>
-		    <origin rpy="0 0 0" xyz="0 0 0" />
-		    <geometry>
-		        <mesh filename="${mesh_dir}/m0609_collision/MF0609_2_1.dae" scale="0.001 0.001 0.001" />
-		    </geometry>
-		</collision>
-		<visual>
-		    <origin rpy="0 0 0" xyz="0 0 0" />
-		    <geometry>
-		        <mesh filename="${mesh_dir}/m0609_white/MF0609_2_1.dae" scale="0.001 0.001 0.001" />
-		    </geometry>
-		</visual>
-		<collision>
-		    <origin rpy="0 0 0" xyz="0 0 0" />
-		    <geometry>
-		        <mesh filename="${mesh_dir}/m0609_collision/MF0609_2_2.dae" scale="0.001 0.001 0.001" />
-		    </geometry>
-		</collision>
-		<visual>
-		    <origin rpy="0 0 0" xyz="0 0 0" />
-		    <geometry>
-		        <mesh filename="${mesh_dir}/m0609_white/MF0609_2_2.dae" scale="0.001 0.001 0.001" />
-		    </geometry>
-		</visual>
-	    </link>
-	    <!-- Joint 3 -->
-	    <joint name="joint_3" type="revolute">
-		<parent link="link_2" />
-		<child link="link_3" />
-		<origin rpy="0 0 1.571" xyz="0.411 0 0" />
-		<axis xyz="0 0 1" />
-		<limit effort="5400" lower="-2.618" upper="2.618" velocity="3.1416"/>
-		<dynamics friction="0.3" damping="300.0" stiffness="8000.0"/>
-	    </joint>
-	    <!-- Link 3 -->
-	    <link name="link_3">
-		<inertial>
-		    <mass value="3.6"/>
-		    <origin xyz="-2.2e-05 -0.006867 0.043445"/>
-		    <inertia ixx="0.018342" ixy="1.1302e-05" ixz="-4.5308e-06" iyy="0.018239" iyz="-0.00099247" izz="0.01326"/>
-		</inertial>
-		<collision>
-		    <origin rpy="0 0 0" xyz="0 0 0" />
-		    <geometry>
-		        <mesh filename="${mesh_dir}/m0609_collision/MF0609_3_0.dae" scale="0.001 0.001 0.001" />
-		    </geometry>
-		</collision>
-		<visual>
-		    <origin rpy="0 0 0" xyz="0 0 0" />
-		    <geometry>
-		        <mesh filename="${mesh_dir}/m0609_white/MF0609_3_0.dae" scale="0.001 0.001 0.001" />
-		    </geometry>
-		</visual>
-	    </link>
-	    <!-- Joint 4 -->
-	    <joint name="joint_4" type="revolute">
-		<parent link="link_3" />
-		<child link="link_4" />
-		<origin rpy="1.571 0 0" xyz="0 -0.368 0" />
-		<axis xyz="0 0 1" />
-		<limit effort="2700" lower="-6.2832" upper="6.2832" velocity="3.927"/>
-		<dynamics friction="0.2" damping="150.0" stiffness="5000.0"/>
-	    </joint>
-	    <!-- Link 4 -->
-	    <link name="link_4">
-		<inertial>
-		    <mass value="3.57"/>
-		    <origin xyz="4e-05 0.097079 -0.10981"/>
-		    <inertia ixx="0.08035" ixy="-4.6119e-06" ixz="-8.1798e-06" iyy="0.066005" iyz="-0.028996" izz="0.029763"/>
-		</inertial>
-		<collision>
-		    <origin rpy="0 0 0" xyz="0 0 0" />
-		    <geometry>
-		        <mesh filename="${mesh_dir}/m0609_collision/MF0609_4_0.dae" scale="0.001 0.001 0.001" />
-		    </geometry>
-		</collision>
-		<visual>
-		    <origin rpy="0 0 0" xyz="0 0 0" />
-		    <geometry>
-		        <mesh filename="${mesh_dir}/m0609_white/MF0609_4_0.dae" scale="0.001 0.001 0.001" />
-		    </geometry>
-		</visual>
-		<collision>
-		    <origin rpy="0 0 0" xyz="0 0 0" />
-		    <geometry>
-		        <mesh filename="${mesh_dir}/m0609_collision/MF0609_4_1.dae" scale="0.001 0.001 0.001" />
-		    </geometry>
-		</collision>
-		<visual>
-		    <origin rpy="0 0 0" xyz="0 0 0" />
-		    <geometry>
-		        <mesh filename="${mesh_dir}/m0609_white/MF0609_4_1.dae" scale="0.001 0.001 0.001" />
-		    </geometry>
-		</visual>
-	    </link>
-	    <!-- Joint 5 -->
-	    <joint name="joint_5" type="revolute">
-		<parent link="link_4" />
-		<child link="link_5" />
-		<origin rpy="-1.571 0 0" xyz="0 0 0" />
-		<axis xyz="0 0 1" />
-		<limit effort="2700" lower="-6.2832" upper="6.2832" velocity="3.927"/>
-		<dynamics friction="0.2" damping="150.0" stiffness="5000.0"/>
-	    </joint>
-	    <!-- Link 5 -->
-	    <link name="link_5">
-		<inertial>
-		    <mass value="2.83"/>
-		    <origin xyz="-6.8e-05 0.003827 0.031969"/>
-		    <inertia ixx="0.014275" ixy="2.2026e-05" ixz="3.3017e-06" iyy="0.012569" iyz="0.00045077" izz="0.0085318"/>
-		</inertial>
-		<collision>
-		    <origin rpy="0 0 0" xyz="0 0 0" />
-		    <geometry>
-		        <mesh filename="${mesh_dir}/m0609_collision/MF0609_5_0.dae" scale="0.001 0.001 0.001" />
-		    </geometry>
-		</collision>
-		<visual>
-		    <origin rpy="0 0 0" xyz="0 0 0" />
-		    <geometry>
-		        <mesh filename="${mesh_dir}/m0609_white/MF0609_5_0.dae" scale="0.001 0.001 0.001" />
-		    </geometry>
-		</visual>
-	    </link>
-	    <!-- Joint 6 -->
-	    <joint name="joint_6" type="revolute">
-		<parent link="link_5" />
-		<child link="link_6" />
-		<origin rpy="1.571 0 0" xyz="0 -0.121 0" />
-		<axis xyz="0 0 1" />
-		<limit effort="2700" lower="-6.2832" upper="6.2832" velocity="3.927"/>
-		<dynamics friction="0.1" damping="100.0" stiffness="3000.0"/>
-	    </joint>
-	    <!-- Link 6 -->
-	    <link name="link_6">
-		<inertial>
-		    <mass value="1.16"/>
-		    <origin xyz="-3e-05 -4.5e-05 -0.0539"/>
-		    <inertia ixx="0.0080226" ixy="1.371e-06" ixz="6.3578e-06" iyy="0.0053992" iyz="7.4676e-06" izz="0.0053912"/>
-		</inertial>
-		<collision>
-		    <origin rpy="0 0 0" xyz="0 0 0" />
-		    <geometry>
-		        <mesh filename="${mesh_dir}/m0609_collision/MF0609_6_0.dae" scale="0.001 0.001 0.001" />
-		    </geometry>
-		</collision>
-		<visual>
-		    <origin rpy="0 0 0" xyz="0 0 0" />
-		    <geometry>
-		        <mesh filename="${mesh_dir}/m0609_white/MF0609_6_0.dae" scale="0.001 0.001 0.001" />
-		    </geometry>
-		</visual>
-	    </link>
-	    <!-- End-Effector Mounting Link (tool0) -->
-	    <link name="tool0"/>
-	    <joint name="joint_6-tool0" type="fixed">
-		<origin rpy="0 0 0" xyz="0 0 0"/>
-		<parent link="link_6"/>
-		<child link="tool0"/>
-	    </joint>
-	</xacro:macro>
-</robot>
+../../../../../ros2_ws/src/arm_cell/arm_cell_description/urdf/m0609_macro.xacro
